Commit message: update

File: description/robot.urdf.xacro (robot description, xacro)
@@ -1,7 +1,13 @@
 <?xml version="1.0"?>
 <robot xmlns:xacro="http://www.ros.org/wiki/xacro"  name="robot">
+    <xacro:arg name="use_ros2_control" default="true"/>
+    <xacro:arg name="sim_mode" default="true"/>  <!--false for real robot-->
     <xacro:include filename="robot_core.xacro" />
-    <!-- <xacro:include filename="gazebo_control.xacro" /> -->
+    <xacro:if value="$(arg use_ros2_control)">
+        <xacro:include filename="ros2_control.xacro" />
+    </xacro:if>
+    <xacro:unless value="$(arg use_ros2_control)">
+        <xacro:include filename="gazebo_control.xacro" />
+    </xacro:unless>
     <xacro:include filename="lidar.xacro" />
-    <xacro:include filename="ros2_control.xacro" />
 </robot>

File: description/robot_core.xacro (robot description, xacro)
@@ -2,5 +2,14 @@
 <robot xmlns:xacro="http://www.ros.org/wiki/xacro" >
  <xacro:include filename="inertial_macros.xacro" />
-  <material name="white">
+    <xacro:property name="chassis_length" value="0.55"/>
+    <xacro:property name="chassis_width" value="0.4"/>
+    <xacro:property name="chassis_height" value="0.25"/>
+    <xacro:property name="chassis_mass" value="0.5"/>
+    <xacro:property name="wheel_radius" value="0.065"/>
+    <xacro:property name="wheel_thickness" value="0.06"/>
+    <xacro:property name="wheel_mass" value="0.1"/>
+    <xacro:property name="wheel_offset_x" value="0.45"/>
+    <xacro:property name="wheel_offset_y" value="0.2"/>
+<material name="white">
     <color rgba="1 1 1 1"/>
 </material>
@@ -20,4 +29,12 @@
 <link name="base_link">
 </link>
+<!-- BASE_FOOTPRINT LINK -->
+<joint name="base_footprint_joint" type="fixed">
+    <parent link="base_link"/>
+    <child link="base_footprint"/>
+    <origin xyz="0 0 0" rpy="0 0 0"/>
+</joint>
+<link name="base_footprint">
+</link>
 <!-- CHASSIS LINK -->
 <joint name="chasis_joint" type="fixed">
@@ -28,28 +45,28 @@
 <link name="chassis">
     <visual>
-        <origin xyz="0.275 0 0.125" rpy="0 0 0"/>
+        <origin xyz="${chassis_length/2} 0 ${chassis_height/2}" rpy="0 0 0"/>
         <geometry>
-            <box size="0.55 0.4 0.25"/>
+            <box size="${chassis_length} ${chassis_width} ${chassis_height}"/>
         </geometry>
-        <material name="white"/>
+        <material name="blue"/>
     </visual>
     <collision>
-        <origin xyz="0.275 0 0.125" rpy="0 0 0"/>
+        <origin xyz="${chassis_length/2} 0 ${chassis_height/2}" rpy="0 0 0"/>
         <geometry>
-            <box size="0.55 0.4 0.25"/>
+            <box size="${chassis_length} ${chassis_width} ${chassis_height}"/>
         </geometry>
     </collision>
-    <xacro:inertial_box mass="0.5" x="0.55" y="0.4" z="0.25">
-     <origin xyz="0.275 0 0.125" rpy="0 0 0"/>
+    <xacro:inertial_box mass="${chassis_mass}" x="${chassis_length}" y="${chassis_width}" z="${chassis_height}">
+     <origin xyz="${chassis_length/2} 0 ${chassis_height/2}" rpy="0 0 0"/>
     </xacro:inertial_box>
 </link>
-    <gazebo reference="chassis">
-        <material>Gazebo/White</material>
-    </gazebo>
+<gazebo reference="chassis">
+    <material>Gazebo/Blue</material>
+</gazebo>
 <!-- Back LEFT WHEEL -->
 <joint name="back_left_wheel_joint" type="continuous">
     <parent link="base_link"/>
     <child link="back_left_wheel"/>
-    <origin xyz="0 0.2 0" rpy="-${pi/2} 0 0"/>
+    <origin xyz="0 ${wheel_offset_y} 0" rpy="-${pi/2} 0 0"/>
     <axis xyz="0 0 1"/>
 </joint>
@@ -57,25 +74,25 @@
     <visual>
         <geometry>
-            <cylinder length="0.06" radius="0.065" />
+            <cylinder length="${wheel_thickness}" radius="${wheel_radius}" />
         </geometry>
-        <material name="blue"/>
+        <material name="black"/>
     </visual>
     <collision>
         <geometry>
-            <cylinder length="0.06" radius="0.065" />
+            <cylinder length="${wheel_thickness}" radius="${wheel_radius}" />
         </geometry>
     </collision>
-    <xacro:inertial_cylinder mass="0.1" length="0.06" radius="0.065">
+    <xacro:inertial_cylinder mass="${wheel_mass}" length="${wheel_thickness}" radius="${wheel_radius}">
       <origin xyz="0 0 0" rpy="0 0 0"/>
     </xacro:inertial_cylinder>
 </link>
-    <gazebo reference="back_left_wheel">
-        <material>Gazebo/Black</material>
-    </gazebo>
+<gazebo reference="back_left_wheel">
+    <material>Gazebo/Black</material>
+</gazebo>
 <!-- BACK RIGHT WHEEL -->
 <joint name="back_right_wheel_joint" type="continuous">
     <parent link="base_link"/>
     <child link="back_right_wheel"/>
-    <origin xyz="0 -0.2 0" rpy="${pi/2} 0 0"/>
+    <origin xyz="0 ${-wheel_offset_y} 0" rpy="${pi/2} 0 0"/>
     <axis xyz="0 0 -1"/>
 </joint>
@@ -83,25 +100,25 @@
     <visual>
         <geometry>
-            <cylinder length="0.06" radius="0.065" />
+            <cylinder length="${wheel_thickness}" radius="${wheel_radius}" />
         </geometry>
-        <material name="blue"/>
+        <material name="black"/>
     </visual>
     <collision>
         <geometry>
-            <cylinder length="0.06" radius="0.065" />
+            <cylinder length="${wheel_thickness}" radius="${wheel_radius}" />
         </geometry>
     </collision>
-    <xacro:inertial_cylinder mass="0.1" length="0.06" radius="0.065">
+    <xacro:inertial_cylinder mass="${wheel_mass}" length="${wheel_thickness}" radius="${wheel_radius}">
       <origin xyz="0 0 0" rpy="0 0 0"/>
     </xacro:inertial_cylinder>
 </link>
-    <gazebo reference="back_right_wheel">
-        <material>Gazebo/Black</material>
-    </gazebo>
+<gazebo reference="back_right_wheel">
+    <material>Gazebo/Black</material>
+</gazebo>
 <!-- FRONT LEFT WHEEL -->
 <joint name="front_left_wheel_joint" type="fixed">
     <parent link="chassis"/>
     <child link="front_left_wheel"/>
-    <origin xyz="0.45 0.2 0" rpy="-${pi/2} 0 0"/>
+    <origin xyz="${wheel_offset_x} ${wheel_offset_y} 0" rpy="-${pi/2} 0 0"/>
     <axis xyz="0 0 1"/>
 </joint>
@@ -109,5 +126,5 @@
     <visual>
         <geometry>
-            <cylinder length="0.06" radius="0.065" />
+            <cylinder length="${wheel_thickness}" radius="${wheel_radius}" />
         </geometry>
         <material name="black"/>
@@ -115,20 +132,20 @@
     <collision>
         <geometry>
-            <cylinder length="0.06" radius="0.065" />
+            <cylinder length="${wheel_thickness}" radius="${wheel_radius}" />
         </geometry>
         <material name="black"/>
     </collision>
-    <xacro:inertial_cylinder mass="0.1" length="0.06" radius="0.065">
+    <xacro:inertial_cylinder mass="${wheel_mass}" length="${wheel_thickness}" radius="${wheel_radius}">
       <origin xyz="0 0 0" rpy="0 0 0"/>
     </xacro:inertial_cylinder>
 </link>
-    <gazebo reference="front_left_wheel">
-        <material>Gazebo/Black</material>
-    </gazebo>
+<gazebo reference="front_left_wheel">
+    <material>Gazebo/Black</material>
+</gazebo>
 <!-- FRONT RIGHT WHEEL -->
 <joint name="front_right_wheel_joint" type="fixed">
     <parent link="chassis"/>
     <child link="front_right_wheel"/>
-    <origin xyz="0.45 -0.2 0" rpy="${pi/2} 0 0"/>
+    <origin xyz="${wheel_offset_x} ${-wheel_offset_y} 0" rpy="${pi/2} 0 0"/>
     <axis xyz="0 0 -1"/>
 </joint>
@@ -136,5 +153,5 @@
     <visual>
         <geometry>
-            <cylinder length="0.06" radius="0.065" />
+         <cylinder length="${wheel_thickness}" radius="${wheel_radius}"/>
         </geometry>
         <material name="black"/>
@@ -142,14 +159,14 @@
     <collision>
         <geometry>
-            <cylinder length="0.06" radius="0.065" />
+            <cylinder length="${wheel_thickness}" radius="${wheel_radius}" />
         </geometry>
         <material name="black"/>
     </collision>
-    <xacro:inertial_cylinder mass="0.1" length="0.06" radius="0.065">
+    <xacro:inertial_cylinder mass="${wheel_mass}" length="${wheel_thickness}" radius="${wheel_radius}">
       <origin xyz="0 0 0" rpy="0 0 0"/>
     </xacro:inertial_cylinder>
 </link>
-     <gazebo reference="front_right_wheel">
-        <material>Gazebo/Black</material>
-    </gazebo>
+ <gazebo reference="front_right_wheel">
+    <material>Gazebo/Black</material>
+</gazebo>
 </robot>

File: description/ros2_control.xacro (robot description, xacro)
@@ -1,28 +1,61 @@
 <?xml version="1.0"?>
 <robot xmlns:xacro="http://www.ros.org/wiki/xacro">
-    <ros2_control name="GazeboSystem" type="system">
-        <hardware>
-            <plugin>gazebo_ros2_control/GazeboSystem</plugin>
-        </hardware>
-        <joint name="back_left_wheel_joint">
-            <command_interface name="velocity">
-                <param name="min">-10</param>
-                <param name="max">10</param>
-            </command_interface>
-            <state_interface name="velocity"/>
-            <state_interface name="position"/>
-        </joint>
-        <joint name="back_right_wheel_joint">
-            <command_interface name="velocity">
-                <param name="min">-10</param>
-                <param name="max">10</param>
-            </command_interface>
-            <state_interface name="velocity"/>
-            <state_interface name="position"/>
-        </joint>
-    </ros2_control>
+    <xacro:unless value="$(arg sim_mode)">
+        <ros2_control name="RealRobot" type="system">
+            <hardware>
+                <plugin>diffdrive_arduino/DiffDriveArduino</plugin>
+                <param name="back_left_wheel_name">back_left_wheel_joint</param>
+                <param name="back_right_wheel_name">back_right_wheel_joint</param>
+                <param name="loop_rate">30</param>
+                <param name="device">/dev/ttyUSB0</param>
+                <param name="baud_rate">57600</param>
+                <param name="timeout">1000</param>
+                <param name="enc_counts_per_rev">3436</param>
+            </hardware>
+            <joint name="back_left_wheel_joint">
+                <command_interface name="velocity">
+                    <param name="min">-10</param>
+                    <param name="max">10</param>
+                </command_interface>
+                <state_interface name="velocity"/>
+                <state_interface name="position"/>
+            </joint>
+            <joint name="back_right_wheel_joint">
+                <command_interface name="velocity">
+                    <param name="min">-10</param>
+                    <param name="max">10</param>
+                </command_interface>
+                <state_interface name="velocity"/>
+                <state_interface name="position"/>
+            </joint>
+        </ros2_control>
+    </xacro:unless>
+    <xacro:if value="$(arg sim_mode)">
+        <ros2_control name="GazeboSystem" type="system">
+            <hardware>
+                <plugin>gazebo_ros2_control/GazeboSystem</plugin>
+            </hardware>
+            <joint name="back_left_wheel_joint">
+                <command_interface name="velocity">
+                    <param name="min">-10</param>
+                    <param name="max">10</param>
+                </command_interface>
+                <state_interface name="velocity"/>
+                <state_interface name="position"/>
+            </joint>
+            <joint name="back_right_wheel_joint">
+                <command_interface name="velocity">
+                    <param name="min">-10</param>
+                    <param name="max">10</param>
+                </command_interface>
+                <state_interface name="velocity"/>
+                <state_interface name="position"/>
+            </joint>
+        </ros2_control>
+    </xacro:if>
     <gazebo>
         <plugin name="gazebo_ros2_control" filename="libgazebo_ros2_control.so">
             <parameters>$(find my_bot)/config/my_controllers.yaml</parameters>
+            <parameters>$(find my_bot)/config/gaz_ros2_ctl_use_sim.yaml</parameters>
         </plugin>
     </gazebo>
